File: hw/power.kicad_sch (KiCad schematic)
At the start: 14 parts, among them U3 MIC2288, U4 LD1117S33TR_SOT223, U5 LD1117S33TR_SOT223

Commit message: Updates to silicon-toaster for components you can buy
Parts:
- U3: ManufacturerRef MBRM140T3G -> MIC2288YD5-TR
